Commit message: configured go1 related file

File: legged_perceptive_description/urdf/robot.xacro (robot description, xacro)
@@ -4,17 +4,17 @@
     <xacro:include filename="$(find legged_unitree_description)/urdf/robot.xacro"/>
     <xacro:include filename="$(find legged_perceptive_description)/urdf/sensor_d435.xacro"/>
-    <xacro:include filename="$(find legged_perceptive_description)/urdf/sensor_t265.xacro"/>
-    <xacro:include filename="$(find legged_perceptive_description)/urdf/mid360.xacro"/>
-    <!--    <xacro:sensor_d435 name="front_camera" topics_ns="front_camera" parent="base">-->
-    <!--        <origin xyz="0.36 -0.0 0.01" rpy="3.141 0.38 0"/>-->
-    <!--    </xacro:sensor_d435>-->
-    <xacro:sensor_t265 name="tracking_camera" topics_ns="tracking_camera" parent="base">
+    <!-- <xacro:include filename="$(find legged_perceptive_description)/urdf/sensor_t265.xacro"/> -->
+    <!-- <xacro:include filename="$(find legged_perceptive_description)/urdf/mid360.xacro"/> -->
+       <xacro:sensor_d435 name="front_camera" topics_ns="front_camera" parent="base">
+           <origin xyz="0.31 -0.0 0.11" rpy="3.141 0.38 0"/>
+       </xacro:sensor_d435>
+    <!-- <xacro:sensor_t265 name="tracking_camera" topics_ns="tracking_camera" parent="base">
         <origin xyz="0.16 0 0.085" rpy="0 -1.04 0"/>
-    </xacro:sensor_t265>
-    <xacro:mid360 name="livox_right" parent="base">
+    </xacro:sensor_t265> -->
+    <!-- <xacro:mid360 name="livox_right" parent="base">
         <origin xyz="0.365 -0.068 -0.030" rpy="-2.59 1.03 3.09"/>
     </xacro:mid360>
     <xacro:mid360 name="livox_left" parent="base">
         <origin xyz="0.365 0.068 -0.030" rpy="2.59 1.03 -3.09"/>
-    </xacro:mid360>
+    </xacro:mid360> -->
 </robot>
